Commit message: TROT GAIT 26.01.06

File: src/robots/go2_descriptions/urdf/go2.urdf (robot description, URDF)
Before this commit: robot go2, 29 links, 28 joints
Links:
- link FL_calf: geometry collision cylinder length=0.12 radius=0.012; visual mesh filename=$(find go2_descriptions)/go2/meshes/calf.dae
- link FL_foot: geometry collision sphere radius=0.022; visual mesh filename=$(find go2_descriptions)/go2/meshes/foot.dae
- link FL_hip: geometry collision cylinder length=0.04 radius=0.046; visual mesh filename=$(find go2_descriptions)/go2/meshes/hip.dae
- link FL_thigh: geometry collision box size=0.213 0.0245 0.034; visual mesh filename=$(find go2_descriptions)/go2/meshes/thigh.dae
- link FR_calf: geometry collision cylinder length=0.12 radius=0.013; visual mesh filename=$(find go2_descriptions)/go2/meshes/calf_mirror.dae
- link FR_foot: geometry collision sphere radius=0.022; visual mesh filename=$(find go2_descriptions)/go2/meshes/foot.dae
- link FR_hip: geometry collision cylinder length=0.04 radius=0.046; visual mesh filename=$(find go2_descriptions)/go2/meshes/hip.dae
- link FR_thigh: geometry collision box size=0.213 0.0245 0.034; visual mesh filename=$(find go2_descriptions)/go2/meshes/thigh_mirror.dae
- link RL_calf: geometry collision cylinder length=0.12 radius=0.013; visual mesh filename=$(find go2_descriptions)/go2/meshes/calf.dae
- link RL_foot: geometry collision sphere radius=0.022; visual mesh filename=$(find go2_descriptions)/go2/meshes/foot.dae
- link RL_hip: geometry collision cylinder length=0.04 radius=0.046; visual mesh filename=$(find go2_descriptions)/go2/meshes/hip.dae
- link RL_thigh: geometry collision box size=0.213 0.0245 0.034; visual mesh filename=$(find go2_descriptions)/go2/meshes/thigh.dae
- link RR_calf: geometry collision cylinder length=0.12 radius=0.013; visual mesh filename=$(find go2_descriptions)/go2/meshes/calf_mirror.dae
- link RR_foot: geometry collision sphere radius=0.022; visual mesh filename=$(find go2_descriptions)/go2/meshes/foot.dae
- link RR_hip: geometry collision cylinder length=0.04 radius=0.046; visual mesh filename=$(find go2_descriptions)/go2/meshes/hip.dae
- link RR_thigh: geometry collision box size=0.213 0.0245 0.034; visual mesh filename=$(find go2_descriptions)/go2/meshes/thigh_mirror.dae
- link base: geometry collision box size=0.3762 0.0935 0.114; visual mesh filename=$(find go2_descriptions)/go2/meshes/base.dae

File: src/robots/go2_descriptions/urdf/go2.xacro (robot description, xacro)
@@ -827,7 +827,8 @@
     </plugin>
   </gazebo>
+  <!-- 지면과의 마찰 및 착지 인식 알고리즘 -->
   <gazebo reference="FL_foot">
-    <mu1>0.3</mu1>
-    <mu2>0.3</mu2>
+    <mu1>0.8</mu1>
+    <mu2>0.8</mu2>
     <self_collide>1</self_collide>
     <material>Gazebo/DarkGrey</material>
@@ -838,5 +839,5 @@
       <update_rate>1000</update_rate>
       <contact>
-        <collision>FL_calf_fixed_joint_lump__FL_foot_collision_1</collision>
+        <collision>FL_calf_fixed_joint_lump__FL_foot_collision_3</collision>
       </contact>
       <plugin name="FL_contact_plugin" filename="libgazebo_ros_bumper.so">
@@ -847,6 +848,6 @@
   </gazebo>
   <gazebo reference="FR_foot">
-    <mu1>0.3</mu1>
-    <mu2>0.3</mu2>
+    <mu1>0.8</mu1>
+    <mu2>0.8</mu2>
     <self_collide>1</self_collide>
     <material>Gazebo/DarkGrey</material>
@@ -857,5 +858,5 @@
       <update_rate>1000</update_rate>
       <contact>
-        <collision>FR_calf_fixed_joint_lump__FR_foot_collision_1</collision>
+        <collision>FR_calf_fixed_joint_lump__FR_foot_collision_3</collision>
       </contact>
       <plugin name="FR_contact_plugin" filename="libgazebo_ros_bumper.so">
@@ -866,6 +867,6 @@
   </gazebo>
   <gazebo reference="RL_foot">
-    <mu1>0.3</mu1>
-    <mu2>0.3</mu2>
+    <mu1>0.8</mu1>
+    <mu2>0.8</mu2>
     <self_collide>1</self_collide>
     <material>Gazebo/DarkGrey</material>
@@ -876,5 +877,5 @@
       <update_rate>1000</update_rate>
       <contact>
-        <collision>RL_calf_fixed_joint_lump__RL_foot_collision_1</collision>
+        <collision>RL_calf_fixed_joint_lump__RL_foot_collision_3</collision>
       </contact>
       <plugin name="RL_contact_plugin" filename="libgazebo_ros_bumper.so">
@@ -885,6 +886,6 @@
   </gazebo>
   <gazebo reference="RR_foot">
-    <mu1>0.3</mu1>
-    <mu2>0.3</mu2>
+    <mu1>0.8</mu1>
+    <mu2>0.8</mu2>
     <self_collide>1</self_collide>
     <material>Gazebo/DarkGrey</material>
@@ -895,5 +896,5 @@
       <update_rate>1000</update_rate>
       <contact>
-        <collision>RR_calf_fixed_joint_lump__RR_foot_collision_1</collision>
+        <collision>RR_calf_fixed_joint_lump__RR_foot_collision_3</collision>
       </contact>
       <plugin name="RR_contact_plugin" filename="libgazebo_ros_bumper.so">
