Commit message: Forward_Kinematics

File: src/robots/go2_descriptions/urdf/go2.xacro (robot description, xacro)
@@ -21,13 +21,14 @@
     <visual>
       <origin xyz="0 0 0" rpy="0 0 0" />
-      <geometry>
-        <mesh filename="package://go2_descriptions/meshes/base.dae" />
-      </geometry>
-      <material name="深色橡胶_001-effect"><color rgba="0.6717055 0.6924257 0.7742702 1" /></material><material name="白色logo_001-effect"><color rgba="1 1 1 1" /></material><material name="黑色贴纸_007-effect"><color rgba="0.009018 0.009018 0.009018 1" /></material><material name="黑色金属_007-effect"><color rgba="0.01341 0.01341 0.01341 1" /></material><material name="黑色塑料_003-effect"><color rgba="0.023455 0.023455 0.023455 1" /></material></visual>
+      <geometry> <mesh filename="package://go2_descriptions/meshes/base.dae" /> </geometry>
+      <material name="深色橡胶_001-effect"><color rgba="0.6717055 0.6924257 0.7742702 1" /></material>
+      <material name="白色logo_001-effect"><color rgba="1 1 1 1" /></material>
+      <material name="黑色贴纸_007-effect"><color rgba="0.009018 0.009018 0.009018 1" /></material>
+      <material name="黑色金属_007-effect"><color rgba="0.01341 0.01341 0.01341 1" /></material>
+      <material name="黑色塑料_003-effect"><color rgba="0.023455 0.023455 0.023455 1" /></material>
+    </visual>
     <collision>
       <origin rpy="0 0 0" xyz="0 0 0" />
-      <geometry>
-        <box size="0.3762 0.0935 0.114" />
-      </geometry>
+      <geometry> <box size="0.3762 0.0935 0.114" /> </geometry>
     </collision>
   </link>
@@ -94,5 +95,5 @@
     <child link="FL_hip" />
     <axis xyz="1 0 0" />
-    <limit lower="-1.0472" upper="1.0472" effort="23.7" velocity="30.1" />
+    <limit lower="-1.0472" upper="1.0472" effort="23.7" velocity="30.1" /> <!-- 이 이상으로 넘어가지 말아라-->
   </joint>
   <link name="FL_hip_rotor">

Commit message: TaskSpacePDControl (2)

File: src/robots/go2_descriptions/urdf/go2.xacro (robot description, xacro)
@@ -82,5 +82,6 @@
         <mesh filename="package://go2_descriptions/meshes/hip.dae" />
       </geometry>
-      <material name="深色橡胶_001-effect"><color rgba="0.6717055 0.6924257 0.7742702 1" /></material><material name="Material-effect"><color rgba="0.9 0.95 0.95 1" /></material></visual>
+      <material name="深色橡胶_001-effect"><color rgba="0.6717055 0.6924257 0.7742702 1" /></material><material name="Material-effect"><color rgba="0.9 0.95 0.95 1" /></material>
+    </visual>
     <collision>
       <origin rpy="1.5707963267948966 0 0" xyz="0 0.08 0" />
@@ -120,5 +121,6 @@
         <mesh filename="package://go2_descriptions/meshes/thigh.dae" />
       </geometry>
-      <material name="深色橡胶_003-effect"><color rgba="0.6717055 0.6924257 0.7742702 1" /></material><material name="Material_009-effect"><color rgba="0.9 0.95 0.95 1" /></material></visual>
+      <material name="深色橡胶_003-effect"><color rgba="0.6717055 0.6924257 0.7742702 1" /></material><material name="Material_009-effect"><color rgba="0.9 0.95 0.95 1" /></material>
+    </visual>
     <collision>
       <origin rpy="0 1.5707963267948966 0" xyz="0 0 -0.1065" />
@@ -158,5 +160,6 @@
         <mesh filename="package://go2_descriptions/meshes/calf.dae" />
       </geometry>
-      <material name="黑色足端_005-effect"><color rgba="0 0 0 1" /></material><material name="深色橡胶_005-effect"><color rgba="0.6717055 0.6924257 0.7742702 1" /></material></visual>
+      <material name="黑色足端_005-effect"><color rgba="0 0 0 1" /></material><material name="深色橡胶_005-effect"><color rgba="0.6717055 0.6924257 0.7742702 1" /></material>
+    </visual>
     <collision>
       <origin rpy="0 -0.21 0" xyz="0.008 0 -0.06" />
@@ -224,5 +227,6 @@
         <mesh filename="package://go2_descriptions/meshes/foot.dae" />
       </geometry>
-      <material name="黑色足端_007-effect"><color rgba="0 0 0 1" /></material></visual>
+      <material name="黑色足端_007-effect"><color rgba="0 0 0 1" /></material>
+    </visual>
     <collision>
       <origin rpy="0 0 0" xyz="-0.002 0 0" />
@@ -249,5 +253,6 @@
         <mesh filename="package://go2_descriptions/meshes/hip.dae" />
       </geometry>
-      <material name="深色橡胶_001-effect"><color rgba="0.6717055 0.6924257 0.7742702 1" /></material><material name="Material-effect"><color rgba="0.9 0.95 0.95 1" /></material></visual>
+      <material name="深色橡胶_001-effect"><color rgba="0.6717055 0.6924257 0.7742702 1" /></material><material name="Material-effect"><color rgba="0.9 0.95 0.95 1" /></material>
+    </visual>
     <collision>
       <origin rpy="1.5707963267948966 0 0" xyz="0 -0.08 0" />
@@ -287,5 +292,6 @@
         <mesh filename="package://go2_descriptions/meshes/thigh_mirror.dae" />
       </geometry>
-      <material name="深色橡胶_012-effect"><color rgba="0.6717055 0.6924257 0.7742702 1" /></material><material name="Material_011-effect"><color rgba="0.9 0.95 0.95 1" /></material></visual>
+      <material name="深色橡胶_012-effect"><color rgba="0.6717055 0.6924257 0.7742702 1" /></material><material name="Material_011-effect"><color rgba="0.9 0.95 0.95 1" /></material>
+    </visual>
     <collision>
       <origin rpy="0 1.5707963267948966 0" xyz="0 0 -0.1065" />
@@ -325,5 +331,6 @@
         <mesh filename="package://go2_descriptions/meshes/calf_mirror.dae" />
       </geometry>
-      <material name="黑色足端_006-effect"><color rgba="0 0 0 1" /></material><material name="深色橡胶_007-effect"><color rgba="0.6717055 0.6924257 0.7742702 1" /></material></visual>
+      <material name="黑色足端_006-effect"><color rgba="0 0 0 1" /></material><material name="深色橡胶_007-effect"><color rgba="0.6717055 0.6924257 0.7742702 1" /></material>
+    </visual>
     <collision>
       <origin rpy="0 -0.2 0" xyz="0.01 0 -0.06" />
@@ -391,5 +398,6 @@
         <mesh filename="package://go2_descriptions/meshes/foot.dae" />
       </geometry>
-      <material name="黑色足端_007-effect"><color rgba="0 0 0 1" /></material></visual>
+      <material name="黑色足端_007-effect"><color rgba="0 0 0 1" /></material>
+    </visual>
     <collision>
       <origin rpy="0 0 0" xyz="-0.002 0 0" />
@@ -416,5 +424,6 @@
         <mesh filename="package://go2_descriptions/meshes/hip.dae" />
       </geometry>
-      <material name="深色橡胶_001-effect"><color rgba="0.6717055 0.6924257 0.7742702 1" /></material><material name="Material-effect"><color rgba="0.9 0.95 0.95 1" /></material></visual>
+      <material name="深色橡胶_001-effect"><color rgba="0.6717055 0.6924257 0.7742702 1" /></material><material name="Material-effect"><color rgba="0.9 0.95 0.95 1" /></material>
+    </visual>
     <collision>
       <origin rpy="1.5707963267948966 0 0" xyz="0 0.08 0" />
@@ -454,5 +463,6 @@
         <mesh filename="package://go2_descriptions/meshes/thigh.dae" />
       </geometry>
-      <material name="深色橡胶_003-effect"><color rgba="0.6717055 0.6924257 0.7742702 1" /></material><material name="Material_009-effect"><color rgba="0.9 0.95 0.95 1" /></material></visual>
+      <material name="深色橡胶_003-effect"><color rgba="0.6717055 0.6924257 0.7742702 1" /></material><material name="Material_009-effect"><color rgba="0.9 0.95 0.95 1" /></material>
+    </visual>
     <collision>
       <origin rpy="0 1.5707963267948966 0" xyz="0 0 -0.1065" />
@@ -492,5 +502,6 @@
         <mesh filename="package://go2_descriptions/meshes/calf.dae" />
       </geometry>
-      <material name="黑色足端_005-effect"><color rgba="0 0 0 1" /></material><material name="深色橡胶_005-effect"><color rgba="0.6717055 0.6924257 0.7742702 1" /></material></visual>
+      <material name="黑色足端_005-effect"><color rgba="0 0 0 1" /></material><material name="深色橡胶_005-effect"><color rgba="0.6717055 0.6924257 0.7742702 1" /></material>
+    </visual>
     <collision>
       <origin rpy="0 -0.2 0" xyz="0.01 0 -0.06" />
@@ -558,5 +569,6 @@
         <mesh filename="package://go2_descriptions/meshes/foot.dae" />
       </geometry>
-      <material name="黑色足端_007-effect"><color rgba="0 0 0 1" /></material></visual>
+      <material name="黑色足端_007-effect"><color rgba="0 0 0 1" /></material>
+    </visual>
     <collision>
       <origin rpy="0 0 0" xyz="-0.002 0 0" />
@@ -583,5 +595,6 @@
         <mesh filename="package://go2_descriptions/meshes/hip.dae" />
       </geometry>
-      <material name="深色橡胶_001-effect"><color rgba="0.6717055 0.6924257 0.7742702 1" /></material><material name="Material-effect"><color rgba="0.9 0.95 0.95 1" /></material></visual>
+      <material name="深色橡胶_001-effect"><color rgba="0.6717055 0.6924257 0.7742702 1" /></material><material name="Material-effect"><color rgba="0.9 0.95 0.95 1" /></material>
+    </visual>
     <collision>
       <origin rpy="1.5707963267948966 0 0" xyz="0 -0.08 0" />

Commit message: TaskSpacePDControl End, SRBM (1)

File: src/robots/go2_descriptions/urdf/go2.xacro (robot description, xacro)
@@ -17,5 +17,5 @@
       <origin xyz="0.021112 0 -0.005366" rpy="0 0 0" />
       <mass value="6.921" />
-      <inertia ixx="0.02448" ixy="0.00012166" ixz="0.0014849" iyy="0.098077" iyz="-3.12E-05" izz="0.107" />
+      <inertia ixx="0.02448" ixy="0.00012166" ixz="0.0014849" iyy="0.098077" iyz="-3.12E-05" izz="0.107" /> <!-- 관성텐서는 서로 대칭 Ixy= Iyx-->
     </inertial>
     <visual>
@@ -634,5 +634,6 @@
         <mesh filename="package://go2_descriptions/meshes/thigh_mirror.dae" />
       </geometry>
-      <material name="深色橡胶_012-effect"><color rgba="0.6717055 0.6924257 0.7742702 1" /></material><material name="Material_011-effect"><color rgba="0.9 0.95 0.95 1" /></material></visual>
+      <material name="深色橡胶_012-effect"><color rgba="0.6717055 0.6924257 0.7742702 1" /></material><material name="Material_011-effect"><color rgba="0.9 0.95 0.95 1" /></material>
+    </visual>
     <collision>
       <origin rpy="0 1.5707963267948966 0" xyz="0 0 -0.1065" />
@@ -672,5 +673,6 @@
         <mesh filename="package://go2_descriptions/meshes/calf_mirror.dae" />
       </geometry>
-      <material name="黑色足端_006-effect"><color rgba="0 0 0 1" /></material><material name="深色橡胶_007-effect"><color rgba="0.6717055 0.6924257 0.7742702 1" /></material></visual>
+      <material name="黑色足端_006-effect"><color rgba="0 0 0 1" /></material><material name="深色橡胶_007-effect"><color rgba="0.6717055 0.6924257 0.7742702 1" /></material>
+    </visual>
     <collision>
       <origin rpy="0 -0.2 0" xyz="0.01 0 -0.06" />
@@ -738,5 +740,6 @@
         <mesh filename="package://go2_descriptions/meshes/foot.dae" />
       </geometry>
-      <material name="黑色足端_007-effect"><color rgba="0 0 0 1" /></material></visual>
+      <material name="黑色足端_007-effect"><color rgba="0 0 0 1" /></material>
+    </visual>
     <collision>
       <origin rpy="0 0 0" xyz="-0.002 0 0" />

Commit message: SRBM_DEBUGING(1)

File: src/robots/go2_descriptions/urdf/go2.xacro (robot description, xacro)
@@ -7,10 +7,10 @@
   <xacro:property name="damping"  value="0.1"/>
   <xacro:property name="friction" value="0.1"/>
-  <link name="world"/>
+  <!-- <link name="world"/>
     <joint name="world_fixed" type="fixed">
       <parent link="world" />
       <child link="base" />
       <origin xyz="0.0 0.0 0.0" rpy="0 0 0" />
-    </joint>
+    </joint> -->
   <link name="base">
     <inertial>
@@ -135,5 +135,5 @@
     <child link="FL_thigh" />
     <axis xyz="0 1 0" />
-    <limit lower="-1.5708" upper="3.4907" effort="23.7" velocity="30.1" />
+    <limit lower="-1.5708" upper="1.5707" effort="23.7" velocity="30.1" />
   </joint>
   <link name="FL_thigh_rotor">
@@ -306,5 +306,5 @@
     <child link="FR_thigh" />
     <axis xyz="0 1 0" />
-    <limit lower="-1.5708" upper="3.4907" effort="23.7" velocity="30.1" />
+    <limit lower="-1.5708" upper="1.5707" effort="23.7" velocity="30.1" />
   </joint>
   <link name="FR_thigh_rotor">
@@ -477,5 +477,5 @@
     <child link="RL_thigh" />
     <axis xyz="0 1 0" />
-    <limit lower="-0.5236" upper="4.5379" effort="23.7" velocity="30.1" />
+    <limit lower="-1.5708" upper="1.5707" effort="23.7" velocity="30.1" />
   </joint>
   <link name="RL_thigh_rotor">
@@ -648,5 +648,5 @@
     <child link="RR_thigh" />
     <axis xyz="0 1 0" />
-    <limit lower="-0.5236" upper="4.5379" effort="23.7" velocity="30.1" />
+    <limit lower="-1.5708" upper="1.5707" effort="23.7" velocity="30.1" />
   </joint>
   <link name="RR_thigh_rotor">
@@ -817,3 +817,79 @@
     </plugin>
   </gazebo>
+  <gazebo reference="FL_foot">
+    <mu1>0.3</mu1>
+    <mu2>0.3</mu2>
+    <self_collide>1</self_collide>
+    <material>Gazebo/DarkGrey</material>
+    <kp value="1000000.0"/>
+    <kd value="10.0"/>
+    <sensor name='FL_foot_contact' type='contact'>
+      <always_on>true</always_on>
+      <update_rate>1000</update_rate>
+      <contact>
+        <collision>FL_calf_fixed_joint_lump__FL_foot_collision_1</collision>
+      </contact>
+      <plugin name="FL_contact_plugin" filename="libgazebo_ros_bumper.so">
+        <bumperTopicName>FL_contactsensor_state</bumperTopicName>
+        <frameName>world</frameName>
+      </plugin>
+    </sensor>
+  </gazebo>
+  <gazebo reference="FR_foot">
+    <mu1>0.3</mu1>
+    <mu2>0.3</mu2>
+    <self_collide>1</self_collide>
+    <material>Gazebo/DarkGrey</material>
+    <kp value="1000000.0"/>
+    <kd value="10.0"/>
+    <sensor name='FR_foot_contact' type='contact'>
+      <always_on>true</always_on>
+      <update_rate>1000</update_rate>
+      <contact>
+        <collision>FR_calf_fixed_joint_lump__FR_foot_collision_1</collision>
+      </contact>
+      <plugin name="FR_contact_plugin" filename="libgazebo_ros_bumper.so">
+        <bumperTopicName>FR_contactsensor_state</bumperTopicName>
+        <frameName>world</frameName>
+      </plugin>
+    </sensor>
+  </gazebo>
+  <gazebo reference="RL_foot">
+    <mu1>0.3</mu1>
+    <mu2>0.3</mu2>
+    <self_collide>1</self_collide>
+    <material>Gazebo/DarkGrey</material>
+    <kp value="1000000.0"/>
+    <kd value="10.0"/>
+    <sensor name='RL_foot_contact' type='contact'>
+      <always_on>true</always_on>
+      <update_rate>1000</update_rate>
+      <contact>
+        <collision>RL_calf_fixed_joint_lump__RL_foot_collision_1</collision>
+      </contact>
+      <plugin name="RL_contact_plugin" filename="libgazebo_ros_bumper.so">
+        <bumperTopicName>RL_contactsensor_state</bumperTopicName>
+        <frameName>world</frameName>
+      </plugin>
+    </sensor>
+  </gazebo>
+  <gazebo reference="RR_foot">
+    <mu1>0.3</mu1>
+    <mu2>0.3</mu2>
+    <self_collide>1</self_collide>
+    <material>Gazebo/DarkGrey</material>
+    <kp value="1000000.0"/>
+    <kd value="10.0"/>
+    <sensor name='RR_foot_contact' type='contact'>
+      <always_on>true</always_on>
+      <update_rate>1000</update_rate>
+      <contact>
+        <collision>RR_calf_fixed_joint_lump__RR_foot_collision_1</collision>
+      </contact>
+      <plugin name="RR_contact_plugin" filename="libgazebo_ros_bumper.so">
+        <bumperTopicName>RR_contactsensor_state</bumperTopicName>
+        <frameName>world</frameName>
+      </plugin>
+    </sensor>
+  </gazebo>
 </robot>

Commit message: SRBM_TOTAL

File: src/robots/go2_descriptions/urdf/go2.xacro (robot description, xacro)
@@ -7,4 +7,5 @@
   <xacro:property name="damping"  value="0.1"/>
   <xacro:property name="friction" value="0.1"/>
+  <!-- 로봇의 공중부양을 도와주는 코드 (link name이 "world"이기 때문)-->
   <!-- <link name="world"/>
     <joint name="world_fixed" type="fixed">
@@ -13,4 +14,13 @@
       <origin xyz="0.0 0.0 0.0" rpy="0 0 0" />
     </joint> -->
+  <!--
+  pinocchio를 사용할 때, "로봇 트리의 가장 첫 번째 링크(Root)는 질량과 관성 정보가 없어야 한다." 라는
+  KDL 규칙을 지키기 위해서 가상의 관성 정보가 0인 Base_Link를 만든거임.
+  -->
+  <link name="base_link"/>
+  <joint name="base_link_to_base" type="fixed">
+    <parent link="base_link"/>
+    <child link="base"/>
+  </joint>
   <link name="base">
     <inertial>

Commit message: 전진보행 구현중 후진함 ㅋㅋ

File: src/robots/go2_descriptions/urdf/go2.xacro (robot description, xacro)
@@ -107,4 +107,5 @@
     <axis xyz="1 0 0" />
     <limit lower="-1.0472" upper="1.0472" effort="23.7" velocity="30.1" /> <!-- 이 이상으로 넘어가지 말아라-->
+    <dynamics damping="${damping}" friction="${friction}"/>
   </joint>
   <link name="FL_hip_rotor">
@@ -146,4 +147,5 @@
     <axis xyz="0 1 0" />
     <limit lower="-1.5708" upper="1.5707" effort="23.7" velocity="30.1" />
+    <dynamics damping="${damping}" friction="${friction}"/>
   </joint>
   <link name="FL_thigh_rotor">
@@ -185,4 +187,5 @@
     <axis xyz="0 1 0" />
     <limit lower="-2.7227" upper="-0.83776" effort="45.43" velocity="15.70" />
+    <dynamics damping="${damping}" friction="${friction}"/>
   </joint>
   <link name="FL_calflower">
@@ -278,4 +281,5 @@
     <axis xyz="1 0 0" />
     <limit lower="-1.0472" upper="1.0472" effort="23.7" velocity="30.1" />
+    <dynamics damping="${damping}" friction="${friction}"/>
   </joint>
   <link name="FR_hip_rotor">
@@ -317,4 +321,5 @@
     <axis xyz="0 1 0" />
     <limit lower="-1.5708" upper="1.5707" effort="23.7" velocity="30.1" />
+    <dynamics damping="${damping}" friction="${friction}"/>
   </joint>
   <link name="FR_thigh_rotor">
@@ -356,4 +361,5 @@
     <axis xyz="0 1 0" />
     <limit lower="-2.7227" upper="-0.83776" effort="45.43" velocity="15.70" />
+    <dynamics damping="${damping}" friction="${friction}"/>
   </joint>
   <link name="FR_calflower">
@@ -449,4 +455,5 @@
     <axis xyz="1 0 0" />
     <limit lower="-1.0472" upper="1.0472" effort="23.7" velocity="30.1" />
+    <dynamics damping="${damping}" friction="${friction}"/>
   </joint>
   <link name="RL_hip_rotor">
@@ -488,4 +495,5 @@
     <axis xyz="0 1 0" />
     <limit lower="-1.5708" upper="1.5707" effort="23.7" velocity="30.1" />
+    <dynamics damping="${damping}" friction="${friction}"/>
   </joint>
   <link name="RL_thigh_rotor">
@@ -527,4 +535,5 @@
     <axis xyz="0 1 0" />
     <limit lower="-2.7227" upper="-0.83776" effort="45.43" velocity="15.70" />
+    <dynamics damping="${damping}" friction="${friction}"/>
   </joint>
   <link name="RL_calflower">
@@ -620,4 +629,5 @@
     <axis xyz="1 0 0" />
     <limit lower="-1.0472" upper="1.0472" effort="23.7" velocity="30.1" />
+    <dynamics damping="${damping}" friction="${friction}"/>
   </joint>
   <link name="RR_hip_rotor">
@@ -659,4 +669,5 @@
     <axis xyz="0 1 0" />
     <limit lower="-1.5708" upper="1.5707" effort="23.7" velocity="30.1" />
+    <dynamics damping="${damping}" friction="${friction}"/>
   </joint>
   <link name="RR_thigh_rotor">
@@ -698,4 +709,5 @@
     <axis xyz="0 1 0" />
     <limit lower="-2.7227" upper="-0.83776" effort="45.43" velocity="15.70" />
+    <dynamics damping="${damping}" friction="${friction}"/>
   </joint>
   <link name="RR_calflower">
